Commit message: 根据kuka fabric 改写tiangong2pro fabric

File: src/fabrics_sim/models/robots/urdf/tiangong2pro/tiangong2pro.urdf (robot description, URDF)
Before this commit: robot tiangong2pro, 49 links, 48 joints
Links:
- removed link A00
- removed link A01
- removed link A02
- removed link B00
- removed link B01
- removed link B02
- removed link C00
- removed link C01
- removed link C02
- removed link D00
- removed link D01
- removed link D02
- removed link base_link_l
- removed link camera_head_link
- removed link elbow_pitch_l_link
- removed link elbow_yaw_l_link
- removed link head_pitch_link
- removed link head_roll_link
- removed link head_yaw_link
- removed link shoulder_pitch_l_link
- removed link shoulder_roll_l_link
- removed link shoulder_yaw_l_link
- removed link wrist_pitch_l_link
- removed link wrist_roll_l_link
- added link palm_x, mass 0.04
- added link palm_x_neg, mass 0.04
- added link palm_y, mass 0.04
- added link palm_y_neg, mass 0.04
- added link palm_z, mass 0.04
- added link palm_z_neg, mass 0.04
- link A00_R: geometry visual mesh filename=meshes/A00_R.STL
- link A01_R: geometry visual mesh filename=meshes/A01_R.STL
- link A02_R: geometry collision box size=0.05 0.025 0.025; visual mesh filename=meshes/A02_R.STL
- link B00_R: geometry visual mesh filename=meshes/B00_R.STL
- link B01_R: geometry collision box size=0.0250 0.0250 0.0500; visual mesh filename=meshes/B01_R.STL
- link B02_R: geometry collision box size=0.025 0.025 0.05; visual mesh filename=meshes/B02_R.STL
- link C00_R: geometry visual mesh filename=meshes/C00_R.STL
- link C01_R: geometry collision box size=0.02500 0.02500 0.0500; visual mesh filename=meshes/C01_R.STL
- link C02_R: geometry collision box size=0.025 0.025 0.045; visual mesh filename=meshes/C02_R.STL
- link D00_R: geometry visual mesh filename=meshes/D00_R.STL
- link D01_R: geometry collision box size=0.0250 0.0250 0.050; visual mesh filename=meshes/D01_R.STL
- link D02_R: geometry collision box size=0.025 0.025 0.045; visual mesh filename=meshes/D02_R.STL
- link base_link_r: geometry collision box size=0.0674 0.0674 0.1348; visual mesh filename=meshes/base_link_r.STL
- link body_yaw_link: geometry collision box size=0.2825 0.2825 0.4; visual mesh filename=meshes/body_yaw_link.STL
- link camera_body_back_link: geometry visual mesh filename=meshes/camera_body_back_link.STL
- link camera_body_front_link: geometry visual mesh filename=meshes/camera_body_front_link.STL
- link elbow_pitch_r_link: geometry visual mesh filename=meshes/elbow_pitch_r_link.STL
- link elbow_yaw_r_link: geometry collision box size=0.0944 0.0944 0.1887; visual mesh filename=meshes/elbow_yaw_r_link.STL
- link shoulder_pitch_r_link: geometry visual mesh filename=meshes/shoulder_pitch_r_link.STL
- link shoulder_roll_r_link: geometry visual mesh filename=meshes/shoulder_roll_r_link.STL
- link shoulder_yaw_r_link: geometry collision box size=0.0993 0.0993 0.1985; visual mesh filename=meshes/shoulder_yaw_r_link.STL
- link wrist_pitch_r_link: geometry visual mesh filename=meshes/wrist_pitch_r_link.STL
- link wrist_roll_r_link: geometry visual mesh filename=meshes/wrist_roll_r_link.STL
Joints:
- removed joint camera_head_joint
- removed joint elbow_pitch_l_joint
- removed joint elbow_yaw_l_joint
- removed joint head_pitch_joint
- removed joint head_roll_joint
- removed joint head_yaw_joint
- removed joint jointA00
- removed joint jointA01
- removed joint jointA02
- removed joint jointB00
- removed joint jointB01
- removed joint jointB02
- removed joint jointC00
- removed joint jointC01
- removed joint jointC02
- removed joint jointD00
- removed joint jointD01
- removed joint jointD02
- removed joint left_hand_joint
- removed joint shoulder_pitch_l_joint
- removed joint shoulder_roll_l_joint
- removed joint shoulder_yaw_l_joint
- removed joint wrist_pitch_l_joint
- removed joint wrist_roll_l_joint
- added joint palm_x_joint: type fixed, parent base_link_r, child palm_x, origin xyz=0.25 0. 0. rpy=0. 0. 0.
- added joint palm_x_neg_joint: type fixed, parent base_link_r, child palm_x_neg, origin xyz=-0.25 0. 0. rpy=0. 0. 0.
- added joint palm_y_joint: type fixed, parent base_link_r, child palm_y, origin xyz=0. 0.25 0. rpy=0. 0. 0.
- added joint palm_y_neg_joint: type fixed, parent base_link_r, child palm_y_neg, origin xyz=0. -0.25 0. rpy=0. 0. 0.
- added joint palm_z_joint: type fixed, parent base_link_r, child palm_z, origin xyz=0. 0. 0.25 rpy=0. 0. 0.
- added joint palm_z_neg_joint: type fixed, parent base_link_r, child palm_z_neg, origin xyz=0. 0. -0.25 rpy=0. 0. 0.
- joint body_yaw_joint: type revolute -> fixed

Commit message: 修改urdf

File: src/fabrics_sim/models/robots/urdf/tiangong2pro/tiangong2pro.urdf (robot description, URDF)
Before this commit: robot tiangong2pro, 31 links, 30 joints
Joints:
- joint Joint_A01_R: limit lower=0.0 upper=1.0 effort=0.05 velocity=7.5398223686155035 -> lower=0.0 upper=1.5708 effort=0.05 velocity=7.5398223686155035
- joint Joint_A02_R: axis -0.34202 -0.93969 0 -> 0.34202 0.93969 0; limit lower=-1.0 upper=0.0 effort=0.05 velocity=7.5398223686155035 -> lower=0.0 upper=1.5708 effort=0.05 velocity=7.5398223686155035
- joint Joint_B01_R: limit lower=0.0 upper=1.0 effort=0.05 velocity=7.5398223686155035 -> lower=0.0 upper=1.5708 effort=0.05 velocity=7.5398223686155035
- joint Joint_B02_R: axis 0 1 0 -> 0 -1 0; limit lower=-1.0 upper=0.0 effort=0.05 velocity=7.5398223686155035 -> lower=0.0 upper=1.5708 effort=0.05 velocity=7.5398223686155035
- joint Joint_C02_R: axis 0 0.99452 0.10453 -> 0 -0.99452 -0.10453; limit lower=-1.0 upper=0.0 effort=0.05 velocity=7.5398223686155035 -> lower=0.0 upper=1.5708 effort=0.05 velocity=7.5398223686155035
- joint Joint_D02_R: axis 0 0.97237 0.23345 -> 0 -0.97237 -0.23345; limit lower=-1.0 upper=0.0 effort=0.05 velocity=7.5398223686155035 -> lower=0.0 upper=1.5708 effort=0.05 velocity=7.5398223686155035

Commit message: update urdf

File: src/fabrics_sim/models/robots/urdf/tiangong2pro/tiangong2pro.urdf (robot description, URDF)
Before this commit: robot tiangong2pro, 31 links, 30 joints
Links:
- added link camera_head_link, mass 0.1; visual mesh filename=meshes/camera_head_link.STL
- added link head_pitch_link, mass 0.23046; visual mesh filename=meshes/head_pitch_link.STL
- added link head_roll_link, mass 0.844627; collision box size=0.15 0.15 0.2; visual mesh filename=meshes/head_roll_link.STL
- added link head_yaw_link, mass 0.088397; visual mesh filename=meshes/head_yaw_link.STL
- link torso_base_link: geometry collision box size=0.25 0.25 0.924; visual box size=0.25 0.25 0.924
Joints:
- added joint camera_head_joint: type fixed, parent head_roll_link, child camera_head_link, origin xyz=0.075191 0.010935 0.074436 rpy=-1.8326 0 -1.5708, axis 0 0 0
- added joint head_pitch_joint: type fixed, parent head_yaw_link, child head_pitch_link, origin xyz=0.01455 0 0.0304 rpy=0 0.2618 0
- added joint head_roll_joint: type fixed, parent head_pitch_link, child head_roll_link, origin xyz=0 0 0 rpy=0 0 0
- added joint head_yaw_joint: type fixed, parent body_yaw_link, child head_yaw_link, origin xyz=-0.002 0 0.56508 rpy=0 0 0
- joint body_yaw_joint: origin xyz=0 0 1 rpy=0 0 0 -> xyz=0 0 0.924 rpy=0 0 0

Commit message: 修改urdf, 参数,  fabric ,使天工机器人仅仅使用两个手指抓取

File: src/fabrics_sim/models/robots/urdf/tiangong2pro/tiangong2pro.urdf (robot description, URDF)
Before this commit: robot tiangong2pro, 35 links, 34 joints
Joints:
- joint Joint_A00_R: type revolute -> fixed
- joint Joint_A02_R: type revolute -> fixed
- joint Joint_B00_R: type revolute -> fixed
- joint Joint_B02_R: type revolute -> fixed
- joint Joint_C00_R: type revolute -> fixed
- joint Joint_C01_R: type revolute -> fixed
- joint Joint_C02_R: type revolute -> fixed
- joint Joint_D00_R: type revolute -> fixed
- joint Joint_D01_R: type revolute -> fixed
- joint Joint_D02_R: type revolute -> fixed
- joint camera_body_back_joint: axis 0 0 0 -> (none)
- joint camera_body_front_joint: axis 0 0 0 -> (none)
- joint camera_head_joint: axis 0 0 0 -> (none)
