Commit message: 增加掌心球体

File: src/fabrics_sim/models/robots/urdf/tiangong/tiangong2pro.urdf (robot description, URDF)
Before this commit: robot tiangong2pro, 35 links, 34 joints
Links:
- added link base_link_r_sphere
Joints:
- added joint base_link_r_joint_sphere: type fixed, parent base_link_r, child base_link_r_sphere, origin xyz=-0.04 0 -0.07 rpy=0 0 0, axis 0 0 1

Commit message: 修改urdf中的手腕处关节限位

File: src/fabrics_sim/models/robots/urdf/tiangong/tiangong2pro.urdf (robot description, URDF)
Before this commit: robot tiangong2pro, 36 links, 35 joints
Joints:
- joint wrist_pitch_r_joint: limit lower=-1.3089969389957472 upper=1.6580627893946132 effort=6.3 velocity=7.5398223686155035 -> lower=-0.785398163 upper=1.047197551 effort=6.3 velocity=7.5398223686155035
- joint wrist_roll_r_joint: limit lower=-1.309 upper=1.6581 effort=6.3 velocity=7.5398223686155035 -> lower=-1.308996939 upper=1.658062789 effort=6.3 velocity=7.5398223686155035

Commit message: update deps and urdf

File: src/fabrics_sim/models/robots/urdf/tiangong/tiangong2pro.urdf (robot description, URDF)
Before this commit: robot tiangong2pro, 36 links, 35 joints
Joints:
- joint shoulder_roll_r_joint: limit lower=-1.8325957145940461 upper=1.0471975511965976 effort=95.0 velocity=3.979350694547071 -> lower=-2.617993878 upper=0.261799388 effort=95.0 velocity=3.979350694547071
